Commit message: Update podstawy_robotyki.urdf
r2d2

File: podstawy_robotyki.urdf (robot description, URDF)
Before this commit: robot example_robot, 17 links, 16 joints
Links:
- removed link link0_passive
- removed link link0_x_axis
- removed link link1
- removed link link1_passive
- removed link link1_x_axis
- removed link link2
- removed link link2_passive
- removed link link2_x_axis
- removed link link3
- removed link link3_passive
- removed link link3_x_axis
- removed link link4
- removed link link4_passive
- removed link link4_x_axis
- removed link link5
- removed link link5_passive
- removed link link5_x_axis
- added link antenna_link; visual cylinder length=0.05 radius=0.002
- added link base_laser; visual cylinder length=0.07 radius=0.025
- added link base_link; visual box size=0.32 0.26 0.085
- added link cpu_link; visual box size=0.19 0.19 0.07
- added link head_link; visual box size=0.03 0.07 0.11
- added link head_pan_link; visual box size=0.05 0.045 0.045
- added link head_tilt_link; visual box size=0.03 0.038 0.04
- added link left_elbow_link; visual box size=0.035 0.035 0.05
- added link left_hand_link; visual box size=0.03 0.01 0.06
- added link left_lower_arm_link; visual cylinder length=0.11 radius=0.0075
- added link left_shoulder_forward_link; visual box size=0.03 0.05 0.03
- added link left_shoulder_link; visual box size=0.025 0.015 0.05
- added link left_shoulder_up_link; visual box size=0.03 0.05 0.03
- added link left_upper_arm_link; visual cylinder length=0.05 radius=0.0075
- added link left_wrist_link; visual box size=0.03 0.05 0.03
- added link neck_link; visual box size=0.03 0.05 0.042
- added link right_elbow_link; visual box size=0.035 0.035 0.05
- added link right_hand_link; visual box size=0.03 0.01 0.06
- added link right_lower_arm_link; visual cylinder length=0.11 radius=0.0075
- added link right_shoulder_forward_link; visual box size=0.03 0.05 0.03
- added link right_shoulder_link; visual box size=0.025 0.015 0.05
- added link right_shoulder_up_link; visual box size=0.03 0.05 0.03
- added link right_upper_arm_link; visual cylinder length=0.05 radius=0.0075
- added link right_wrist_link; visual box size=0.03 0.05 0.03
- added link torso_link; visual cylinder length=0.24 radius=0.05
- added link upper_base_link; visual cylinder length=0.10 radius=0.085
Joints:
- removed joint q0_x
- removed joint q1
- removed joint q1_passive
- removed joint q1_x
- removed joint q2
- removed joint q2_passive
- removed joint q2_x
- removed joint q3
- removed joint q3_passive
- removed joint q3_x
- removed joint q4
- removed joint q4_passive
- removed joint q4_x
- removed joint q5
- removed joint q5_passive
- removed joint q5_x
- added joint antenna_joint: type fixed, parent head_link, child antenna_link, origin xyz=0.0 -0.025 0.065 rpy=0 0 0
- added joint base_laser_joint: type fixed, parent base_link, child base_laser, origin xyz=0.18 0 0.07 rpy=0 0 0
- added joint cpu_joint: type fixed, parent base_link, child cpu_link, origin xyz=0.025 0 0.085 rpy=0 0 0
- added joint head_pan_joint: type revolute, parent head_pan_link, child head_tilt_link, origin xyz=0 0 0.045 rpy=0 0 0, axis 0 0 1, limit lower=-3.1416 upper=3.1416 effort=10 velocity=3
- added joint head_pan_servo: type fixed, parent torso_link, child head_pan_link, origin xyz=0 0 0.225 rpy=0 0 0
- added joint head_tilt_joint: type revolute, parent head_tilt_link, child neck_link, origin xyz=0 0 0.04 rpy=0 0 0, axis 0 1 0, limit lower=-1.57 upper=1.57 effort=10 velocity=3
- added joint left_elbow_joint: type revolute, parent left_upper_arm_link, child left_elbow_link, origin xyz=-0.005 0 -0.05 rpy=0 0 0, axis 0 0 1, limit lower=-3.146 upper=3.146 effort=10 velocity=3
- added joint left_hand_joint: type fixed, parent left_wrist_link, child left_hand_link, origin xyz=0 0 -0.055 rpy=0 0 0
- added joint left_lower_arm_joint: type fixed, parent left_elbow_link, child left_lower_arm_link, origin xyz=0 0 -0.08 rpy=0 0 0
- added joint left_shoulder_forward_joint: type revolute, parent left_shoulder_link, child left_shoulder_forward_link, origin xyz=0 0.025 0 rpy=0 0 0, axis 0 0 1, limit lower=-1.57 upper=1.57 effort=10 velocity=3
- added joint left_shoulder_joint: type fixed, parent torso_link, child left_shoulder_link, origin xyz=0 0.055 0.165 rpy=0 0 0
- added joint left_shoulder_up_joint: type revolute, parent left_shoulder_forward_link, child left_shoulder_up_link, origin xyz=0 0.04 -0.01 rpy=0 -0.707 0, axis 0 1 0, limit lower=-1.57 upper=1.57 effort=10 velocity=3
- added joint left_upper_arm_joint: type fixed, parent left_shoulder_up_link, child left_upper_arm_link, origin xyz=0 0 -0.05 rpy=0 0 0
- added joint left_wrist_joint: type revolute, parent left_lower_arm_link, child left_wrist_link, origin xyz=0 0 -0.05 rpy=0 0 0, axis 1 0 0, limit lower=-1.57 upper=1.57 effort=10 velocity=3
- added joint neck_joint: type fixed, parent neck_link, child head_link, origin xyz=0.05 0 0.015 rpy=0 0 0
- added joint right_elbow_joint: type revolute, parent right_upper_arm_link, child right_elbow_link, origin xyz=-0.005 0 -0.05 rpy=0 0 0, axis 0 0 1, limit lower=-3.146 upper=3.146 effort=10 velocity=3
- added joint right_hand_joint: type fixed, parent right_wrist_link, child right_hand_link, origin xyz=0 0 -0.055 rpy=0 0 0
- added joint right_lower_arm_joint: type fixed, parent right_elbow_link, child right_lower_arm_link, origin xyz=0 0 -0.08 rpy=0 0 0
- added joint right_shoulder_forward_joint: type revolute, parent right_shoulder_link, child right_shoulder_forward_link, origin xyz=0 -0.025 0 rpy=0 0 0, axis 0 0 1, limit lower=-1.57 upper=1.57 effort=10 velocity=3
- added joint right_shoulder_joint: type fixed, parent torso_link, child right_shoulder_link, origin xyz=0 -0.055 0.165 rpy=0 0 0
- added joint right_shoulder_up_joint: type revolute, parent right_shoulder_forward_link, child right_shoulder_up_link, origin xyz=0 -0.04 -0.01 rpy=0 -0.707 0, axis 0 1 0, limit lower=-1.57 upper=1.57 effort=10 velocity=3
- added joint right_upper_arm_joint: type fixed, parent right_shoulder_up_link, child right_upper_arm_link, origin xyz=0 0 -0.05 rpy=0 0 0
- added joint right_wrist_joint: type revolute, parent right_lower_arm_link, child right_wrist_link, origin xyz=0 0 -0.05 rpy=0 0 0, axis 1 0 0, limit lower=-1.57 upper=1.57 effort=10 velocity=3
- added joint torso_joint: type revolute, parent upper_base_link, child torso_link, origin xyz=0 0 0.10 rpy=0 0 0, axis 0 0 1, limit lower=-3.1416 upper=3.1416 effort=10 velocity=3
- added joint upper_base_joint: type fixed, parent cpu_link, child upper_base_link, origin xyz=0 0 0.07 rpy=0 0 0

Commit message: Update podstawy_robotyki.urdf
back

File: podstawy_robotyki.urdf (robot description, URDF)
Before this commit: robot pi_robot, 26 links, 25 joints
Links:
- removed link antenna_link
- removed link base_laser
- removed link base_link
- removed link cpu_link
- removed link head_link
- removed link head_pan_link
- removed link head_tilt_link
- removed link left_elbow_link
- removed link left_hand_link
- removed link left_lower_arm_link
- removed link left_shoulder_forward_link
- removed link left_shoulder_link
- removed link left_shoulder_up_link
- removed link left_upper_arm_link
- removed link left_wrist_link
- removed link neck_link
- removed link right_elbow_link
- removed link right_hand_link
- removed link right_lower_arm_link
- removed link right_shoulder_forward_link
- removed link right_shoulder_link
- removed link right_shoulder_up_link
- removed link right_upper_arm_link
- removed link right_wrist_link
- removed link torso_link
- removed link upper_base_link
- added link link0_passive; visual origin rpy=0 0 0 xyz=0 0 0
- added link link0_x_axis; visual origin rpy=0 0 0 xyz=0 0 0
- added link link1
- added link link1_passive; visual cylinder length=0.5 radius=0.05
- added link link1_x_axis; visual cylinder length=0.5 radius=0.05
- added link link2
- added link link2_passive; visual cylinder length=0.5 radius=0.05
- added link link2_x_axis; visual cylinder length=0.5 radius=0.05
- added link link3
- added link link3_passive; visual cylinder length=0.5 radius=0.05
- added link link3_x_axis; visual cylinder length=0.5 radius=0.05
- added link link4
- added link link4_passive; visual cylinder length=0.5 radius=0.05
- added link link4_x_axis; visual cylinder length=0.5 radius=0.05
- added link link5
- added link link5_passive; visual cylinder length=0.5 radius=0.05
- added link link5_x_axis; visual cylinder length=0.5 radius=0.05
Joints:
- removed joint antenna_joint
- removed joint base_laser_joint
- removed joint cpu_joint
- removed joint head_pan_joint
- removed joint head_pan_servo
- removed joint head_tilt_joint
- removed joint left_elbow_joint
- removed joint left_hand_joint
- removed joint left_lower_arm_joint
- removed joint left_shoulder_forward_joint
- removed joint left_shoulder_joint
- removed joint left_shoulder_up_joint
- removed joint left_upper_arm_joint
- removed joint left_wrist_joint
- removed joint neck_joint
- removed joint right_elbow_joint
- removed joint right_hand_joint
- removed joint right_lower_arm_joint
- removed joint right_shoulder_forward_joint
- removed joint right_shoulder_joint
- removed joint right_shoulder_up_joint
- removed joint right_upper_arm_joint
- removed joint right_wrist_joint
- removed joint torso_joint
- removed joint upper_base_joint
- added joint q0_x: type fixed, parent link0_passive, child link0_x_axis, origin xyz=0 0 0 rpy=0 1.571 0
- added joint q1: type revolute, parent link0_passive, child link1, origin xyz=0 0 0.815 rpy=0 0 0, axis 0 0 1
- added joint q1_passive: type fixed, parent link1, child link1_passive, origin xyz=0.35 0 0 rpy=1.5707963267948966 0 0
- added joint q1_x: type fixed, parent link1_passive, child link1_x_axis, origin xyz=0 0 0 rpy=0 1.571 0
- added joint q2: type revolute, parent link1_passive, child link2, origin xyz=0 0 0 rpy=0 0 1.5707963267948966, axis 0 0 1
- added joint q2_passive: type fixed, parent link2, child link2_passive, origin xyz=0.85 0 0 rpy=0 0 0
- added joint q2_x: type fixed, parent link2_passive, child link2_x_axis, origin xyz=0 0 0 rpy=0 1.571 0
- added joint q3: type revolute, parent link2_passive, child link3, origin xyz=0 0 0 rpy=0 0 0, axis 0 0 1
- added joint q3_passive: type fixed, parent link3, child link3_passive, origin xyz=0.82 0 0 rpy=1.5707963267948966 0 0
- added joint q3_x: type fixed, parent link3_passive, child link3_x_axis, origin xyz=0 0 0 rpy=0 1.571 0
- added joint q4: type revolute, parent link3_passive, child link4, origin xyz=0 0 0 rpy=0 0 0, axis 0 0 1
- added joint q4_passive: type fixed, parent link4, child link4_passive, origin xyz=0 0 0 rpy=-1.5707963267948966 0 0
- added joint q4_x: type fixed, parent link4_passive, child link4_x_axis, origin xyz=0 0 0 rpy=0 1.571 0
- added joint q5: type revolute, parent link4_passive, child link5, origin xyz=0 0 0.17 rpy=0 0 0, axis 0 0 1
- added joint q5_passive: type fixed, parent link5, child link5_passive, origin xyz=0 0 0 rpy=0 0 0
- added joint q5_x: type fixed, parent link5_passive, child link5_x_axis, origin xyz=0 0 0 rpy=0 1.571 0

Commit message: Add limits to revolute joints

File: podstawy_robotyki.urdf (robot description, URDF)
Before this commit: robot example_robot, 17 links, 16 joints
Links:
- removed link link0_passive
- added link base_link; visual cylinder length=0.0 radius=0.0
- added link link6
- added link link6_passive; visual cylinder length=0.5 radius=0.05
- added link link6_x_axis; visual cylinder length=0.5 radius=0.05
- link link0_x_axis: geometry visual cylinder length=0.0 radius=0.0
Joints:
- added joint q6: type revolute, parent link5_passive, child link6, origin xyz=0 0 0.17 rpy=0 0 0, axis 0 0 1, limit lower=-6.11 upper=6.11 effort=30 velocity=5.61
- added joint q6_passive: type fixed, parent link6, child link6_passive, origin xyz=0 0 0 rpy=0 0 0
- added joint q6_x: type fixed, parent link6_passive, child link6_x_axis, origin xyz=0 0 0 rpy=0 1.571 0
- joint q0_x: parent link0_passive -> base_link
- joint q1: limit (none) -> lower=-3.22 upper=3.22 effort=30 velocity=2.44; parent link0_passive -> base_link
- joint q2: limit (none) -> lower=-2.18 upper=0.79 effort=30 velocity=2.19
- joint q3: limit (none) -> lower=-1.18 upper=0.52 effort=30 velocity=2.44
- joint q3_passive: origin xyz=0.82 0 0 rpy=1.5707963267948966 0 0 -> xyz=0.145 0 0 rpy=1.5707963267948966 0 0
- joint q4: limit (none) -> lower=-6.11 upper=6.11 effort=30 velocity=4.53; origin xyz=0 0 0 rpy=0 0 0 -> xyz=0 0 0.82 rpy=0 0 0
- joint q5: limit (none) -> lower=-2.07 upper=2.07 effort=30 velocity=4.27; origin xyz=0 0 0.17 rpy=0 0 0 -> xyz=0 0 0 rpy=0 0 0
- joint q5_passive: origin xyz=0 0 0 rpy=0 0 0 -> xyz=0 0 0 rpy=1.5707963267948966 0 0

Commit message: Second lecture

File: podstawy_robotyki.urdf (robot description, URDF)
Before this commit: robot KUKA_KR_30-3_R2100, 20 links, 19 joints
Links:
- added link base0; visual cylinder length=0.1 radius=0.35
- added link base1; visual cylinder length=0.795 radius=0.325
- added link base2; visual cylinder length=0.1 radius=0.35

Commit message: Add visualization for last 3 joints

File: podstawy_robotyki.urdf (robot description, URDF)
Before this commit: robot KUKA_KR_30-3_R2100, 20 links, 19 joints
Links:
- removed link link0_x_axis
- removed link link1_x_axis
- removed link link2_x_axis
- removed link link3_x_axis
- removed link link4_x_axis
- removed link link5_x_axis
- removed link link6_passive
- removed link link6_x_axis
- link base_link: geometry visual cylinder length=0.7 radius=0.4
- link link1: geometry visual cylinder length=0.35 radius=0.1
- link link1_passive: geometry 
- link link2_passive: geometry visual cylinder length=0.145 radius=0.05
- link link3_passive: geometry visual cylinder length=0.82 radius=0.05
- link link4_passive: geometry 
- link link5_passive: geometry visual cylinder length=0.17 radius=0.05
- link link6: geometry visual box size=0.1 0.1 0.05
Joints:
- removed joint q0_x
- removed joint q1_x
- removed joint q2_x
- removed joint q3_x
- removed joint q4_x
- removed joint q5_x
- removed joint q6_passive
- removed joint q6_x

Commit message: Fix Link3 visual

File: podstawy_robotyki.urdf (robot description, URDF)
Before this commit: robot KUKA_KR_30-3_R2100, 12 links, 11 joints
Links:
- link link2_passive: geometry 
- link link3: geometry visual cylinder length=0.2 radius=0.05

Commit message: first whole visualization

File: podstawy_robotyki.urdf (robot description, URDF)
Before this commit: robot KUKA_KR_30-3_R2100, 12 links, 11 joints
Links:
- link base_link: geometry visual cylinder length=0.6 radius=0.33
- link link1: geometry 
- link link1_passive: geometry visual box size=0.45 0.2 0.3
- link link2: geometry visual cylinder length=.2 radius=0.1; visual cylinder length=0.8 radius=0.1
- link link2_passive: geometry visual cylinder length=0.2 radius=0.1
- link link3: geometry 
- link link3_passive: geometry visual cylinder length=1 radius=0.05

Commit message: Add q4 joint visualization, cleanup

File: podstawy_robotyki.urdf (robot description, URDF)
Before this commit: robot KUKA_KR_30-3_R2100, 12 links, 11 joints
Links:
- link link4_passive: geometry visual cylinder length=0.11 radius=0.05
